Commit message: code cleanup + imu gz_ros_bridge

File: models/scout_sdf/model.xacro (robot description, xacro)
@@ -2,6 +2,6 @@
 <sdf version="1.10" xmlns:xacro="http://ros.org/wiki/xacro">
 <model name='scout' canonical_link='chassis'>
-  <xacro:property name="update_rate" value="10"/>
-  <xacro:property name="linear_speed" value="1.0"/>
+  <xacro:property name="update_rate"   value="10"/>
+  <xacro:property name="linear_speed"  value="1.0"/>
   <xacro:property name="angular_speed" value="0.5"/>
   <!-- base_link -->
@@ -31,7 +31,8 @@
   </link>
   <!-- wheels -->
-  <xacro:property name="wheel_radius" value="0.16"/>
-  <xacro:property name="wheel_width" value="0.11"/>
-  <xacro:property name="wheel_distance" value="0.29153"/>
+  <xacro:property name="wheel_radius"     value="0.16"/>
+  <xacro:property name="wheel_width"      value="0.11"/>
+  <xacro:property name="wheel_base"       value="0.498"/>
+  <xacro:property name="wheel_separation" value="0.58306"/>
   <xacro:macro name="wheel" params="N T X Y Z r p y">
     <link name='${N}_wheel'>
@@ -68,8 +69,8 @@
     </joint>
   </xacro:macro>
-  <xacro:wheel N='front_left'  T='2' X='0.249'  Y='${wheel_distance}'    Z='-0.0702' r='0.0'   p='0.0' y='0.0'/>
-  <xacro:wheel N='front_right' T='1' X='0.249'  Y='${(-wheel_distance)}' Z='-0.0702' r='${pi}' p='0.0' y='0.0'/>
-  <xacro:wheel N='back_left'   T='1' X='-0.249' Y='${wheel_distance}'    Z='-0.0702' r='0.0'   p='0.0' y='0.0'/>
-  <xacro:wheel N='back_right'  T='2' X='-0.249' Y='${(-wheel_distance)}' Z='-0.0702' r='${pi}' p='0.0' y='0.0'/>
+  <xacro:wheel N='front_left'  T='2' X='${(wheel_base/2)}'  Y='${(wheel_separation/2)}'  Z='-0.0702' r='0.0'   p='0.0' y='0.0'/>
+  <xacro:wheel N='front_right' T='1' X='${(wheel_base/2)}'  Y='${(-wheel_separation/2)}' Z='-0.0702' r='${pi}' p='0.0' y='0.0'/>
+  <xacro:wheel N='back_left'   T='1' X='${(-wheel_base/2)}' Y='${(wheel_separation/2)}'  Z='-0.0702' r='0.0'   p='0.0' y='0.0'/>
+  <xacro:wheel N='back_right'  T='2' X='${(-wheel_base/2)}' Y='${(-wheel_separation/2)}' Z='-0.0702' r='${pi}' p='0.0' y='0.0'/>
   <!-- sensor bar -->
   <xacro:macro name="force_bar_segment" params="P X Y Z r p y L W H">
@@ -124,7 +125,8 @@
     <back_left_joint>back_left_wheel_joint</back_left_joint>
     <back_right_joint>back_right_wheel_joint</back_right_joint>
-    <wheel_separation>${(wheel_distance*2)}</wheel_separation>
+    <wheelbase>${wheel_base}</wheelbase>
+    <wheel_separation>${wheel_separation}</wheel_separation>
     <wheel_radius>${wheel_radius}</wheel_radius>
-    <odom_publish_frequency>${update_rate}</odom_publish_frequency>
+    <odom_publish_frequency>1</odom_publish_frequency>
     <topic>cmd_vel</topic>
   </plugin>
@@ -165,4 +167,12 @@
     <static_update_frequency>${update_rate}</static_update_frequency>
   </plugin>
+  <plugin
+    filename="gz-sim-imu-system"
+    name="gz::sim::systems::Imu">
+  </plugin>
+  <plugin
+    filename="gz-sim-forcetorque-system"
+    name="gz::sim::systems::ForceTorque">
+  </plugin>
 </model>
 </sdf>

Commit message: added simple recording of position

File: models/scout_sdf/model.xacro (robot description, xacro)
@@ -2,7 +2,10 @@
 <sdf version="1.10" xmlns:xacro="http://ros.org/wiki/xacro">
 <model name='scout' canonical_link='chassis'>
-  <xacro:property name="update_rate"   value="10"/>
-  <xacro:property name="linear_speed"  value="1.0"/>
-  <xacro:property name="angular_speed" value="0.5"/>
+  <xacro:property name="update_rate_odom"      value="1"/>
+  <xacro:property name="update_rate_imu"       value="1"/>
+  <xacro:property name="update_rate_pose"      value="3"/>
+  <xacro:property name="update_rate_force_bar" value="100"/>
+  <xacro:property name="linear_speed"          value="1.0"/>
+  <xacro:property name="angular_speed"         value="0.5"/>
   <!-- base_link -->
   <link name='chassis'>
@@ -25,5 +28,5 @@
     <sensor name="imu_sensor" type="imu">
       <always_on>true</always_on>
-      <update_rate>${update_rate}</update_rate>
+      <update_rate>${update_rate_imu}</update_rate>
       <visualize>true</visualize>
       <topic>scout/imu</topic>
@@ -106,5 +109,5 @@
       <sensor name='force_bar_P${P}_sensor' type='force_torque'>
         <always_on>true</always_on>
-        <update_rate>${update_rate}</update_rate>
+        <update_rate>${update_rate_force_bar}</update_rate>
         <visualize>true</visualize>
         <topic>/scout/force_bar/segment_${P}</topic>
@@ -128,5 +131,5 @@
     <wheel_separation>${wheel_separation}</wheel_separation>
     <wheel_radius>${wheel_radius}</wheel_radius>
-    <odom_publish_frequency>1</odom_publish_frequency>
+    <odom_publish_frequency>${update_rate_odom}</odom_publish_frequency>
     <topic>cmd_vel</topic>
   </plugin>
@@ -163,7 +166,7 @@
     <publish_nested_model_pose>True</publish_nested_model_pose>
     <use_pose_vector_msg>False</use_pose_vector_msg>
-    <update_frequency>${update_rate}</update_frequency>
+    <update_frequency>${update_rate_pose}</update_frequency>
     <static_publisher>False</static_publisher>
-    <static_update_frequency>${update_rate}</static_update_frequency>
+    <static_update_frequency>${update_rate_pose}</static_update_frequency>
   </plugin>
   <plugin

Commit message: increased accuracy of bumping

File: models/scout_sdf/model.xacro (robot description, xacro)
@@ -5,6 +5,6 @@
   <xacro:property name="update_rate_imu"       value="1"/>
   <xacro:property name="update_rate_pose"      value="3"/>
-  <xacro:property name="update_rate_force_bar" value="100"/>
-  <xacro:property name="linear_speed"          value="1.0"/>
+  <xacro:property name="update_rate_force_bar" value="1000"/>
+  <xacro:property name="linear_speed"          value="0.5"/>
   <xacro:property name="angular_speed"         value="0.5"/>
   <!-- base_link -->
@@ -90,7 +90,7 @@
         </geometry>
         <material>
-          <ambient>1.0 0.0 0.0 1</ambient>
-          <diffuse>1.0 0.0 0.0 1</diffuse>
-          <specular>1.0 0.0 0.0 1</specular>
+          <ambient>0.5 0.5 0.5 0.5</ambient>
+          <diffuse>0.5 0.5 0.5 0.5</diffuse>
+          <specular>0.5 0.5 0.5 0.5</specular>
         </material>
       </visual>
@@ -115,9 +115,9 @@
     </joint>
   </xacro:macro>
-  <xacro:force_bar_segment P='0' X='0.466' Y='0.28'  Z='-0.025' r='${pi/2}' p='0.0' y='0.43633'  L='0.005' W='0.15' H='0.14'/>
-  <xacro:force_bar_segment P='1' X='0.5'   Y='0.14'  Z='-0.025' r='${pi/2}' p='0.0' y='0.0'      L='0.005' W='0.15' H='0.13'/>
-  <xacro:force_bar_segment P='2' X='0.5'   Y='0.0'   Z='-0.025' r='${pi/2}' p='0.0' y='0.0'      L='0.005' W='0.15' H='0.13'/>
-  <xacro:force_bar_segment P='3' X='0.5'   Y='-0.14' Z='-0.025' r='${pi/2}' p='0.0' y='0.0'      L='0.005' W='0.15' H='0.13'/>
-  <xacro:force_bar_segment P='4' X='0.466' Y='-0.28' Z='-0.025' r='${pi/2}' p='0.0' y='-0.43633' L='0.005' W='0.15' H='0.14'/>
+  <xacro:force_bar_segment P='0' X='0.466' Y='0.28'  Z='0.0' r='${pi/2}' p='0.0' y='0.43633'  L='0.005' W='0.15' H='0.14'/>
+  <xacro:force_bar_segment P='1' X='0.5'   Y='0.14'  Z='0.0' r='${pi/2}' p='0.0' y='0.0'      L='0.005' W='0.15' H='0.13'/>
+  <xacro:force_bar_segment P='2' X='0.5'   Y='0.0'   Z='0.0' r='${pi/2}' p='0.0' y='0.0'      L='0.005' W='0.15' H='0.13'/>
+  <xacro:force_bar_segment P='3' X='0.5'   Y='-0.14' Z='0.0' r='${pi/2}' p='0.0' y='0.0'      L='0.005' W='0.15' H='0.13'/>
+  <xacro:force_bar_segment P='4' X='0.466' Y='-0.28' Z='0.0' r='${pi/2}' p='0.0' y='-0.43633' L='0.005' W='0.15' H='0.14'/>
   <!-- plugins -->
   <plugin

Commit message: pretty simulation part 1

File: models/scout_sdf/model.xacro (robot description, xacro)
@@ -76,4 +76,35 @@
   <xacro:wheel N='back_left'   T='1' X='${(-wheel_base/2)}' Y='${(wheel_separation/2)}'  Z='-0.0702' r='0.0'   p='0.0' y='0.0'/>
   <xacro:wheel N='back_right'  T='2' X='${(-wheel_base/2)}' Y='${(-wheel_separation/2)}' Z='-0.0702' r='${pi}' p='0.0' y='0.0'/>
+  <!-- visual connection -->
+  <xacro:macro name="force_bar_material">
+    <material>
+      <ambient>0.25 0.25 0.25 1.0</ambient>
+      <diffuse>0.25 0.25 0.25 1.0</diffuse>
+      <specular>0.25 0.25 0.25 1.0</specular>
+    </material>
+  </xacro:macro>
+  <xacro:macro name="force_bar_connection_visual" params="N X Y Z r p y L W H">
+    <visual name='force_bar_connection_visual_${N}'>
+      <pose relative_to="chassis">${X} ${Y} ${Z} ${r} ${p} ${y}</pose>
+      <geometry>
+        <box>
+          <size>${L} ${W} ${H}</size>
+        </box>
+      </geometry>
+      <xacro:force_bar_material/>
+    </visual>
+  </xacro:macro>
+  <link name='force_bar_connection_visual'>
+    <xacro:force_bar_connection_visual N='center_bar_left'  X='0.4'    Y='0.04'   Z='0' r='0' p='0' y='0'        L='0.2'   W='0.025' H='0.025'/>
+    <xacro:force_bar_connection_visual N='center_bar_right' X='0.4'    Y='-0.04'  Z='0' r='0' p='0' y='0'        L='0.2'   W='0.025' H='0.025'/>
+    <xacro:force_bar_connection_visual N='front_bar_top'    X='0.4875' Y='0'      Z='0' r='0' p='0' y='0'        L='0.025' W='0.41'  H='0.025'/>
+    <xacro:force_bar_connection_visual N='front_bar_left'   X='0.4575' Y='0.265'  Z='0' r='0' p='0' y='0.43633'  L='0.025' W='0.15'  H='0.025'/>
+    <xacro:force_bar_connection_visual N='front_bar_right'  X='0.4575' Y='-0.265' Z='0' r='0' p='0' y='-0.43633' L='0.025' W='0.15'  H='0.025'/>
+  </link>
+  <joint name='force_bar_connection_visual_joint' type='fixed'>
+    <pose relative_to='force_bar_connection_visual'/>
+    <parent>chassis</parent>
+    <child>force_bar_connection_visual</child>
+  </joint>
   <!-- sensor bar -->
   <xacro:macro name="force_bar_segment" params="P X Y Z r p y L W H">
@@ -89,9 +120,5 @@
           </box>
         </geometry>
-        <material>
-          <ambient>0.5 0.5 0.5 0.5</ambient>
-          <diffuse>0.5 0.5 0.5 0.5</diffuse>
-          <specular>0.5 0.5 0.5 0.5</specular>
-        </material>
+        <xacro:force_bar_material/>
       </visual>
       <collision name='collision'>
