Commit message: bunker pre config

File: src/ros_gz_bunker_lehrforst_sim/models/bunker/model.xacro (robot description, xacro)
@@ -5,5 +5,4 @@
   <xacro:property name="update_rate_imu"       value="1"/>
   <xacro:property name="update_rate_pose"      value="3"/>
-  <xacro:property name="update_rate_force_bar" value="1000"/>
   <xacro:property name="linear_speed"          value="0.5"/>
   <xacro:property name="angular_speed"         value="0.5"/>
@@ -11,152 +10,16 @@
   <link name='chassis'>
     <pose relative_to='__model__'>0 0 1 0 0 0</pose>
-    <inertial auto="true">
-      <mass>50</mass>
-    </inertial>
-    <visual name='visual'>
-      <geometry>
-        <mesh><uri>meshes/scout_base.dae</uri></mesh>
-      </geometry>
-    </visual>
-    <collision name='collision'>
-      <geometry>
-        <box>
-          <size>0.93 0.42 0.19</size>
-        </box>
-      </geometry>
-    </collision>
     <sensor name="imu_sensor" type="imu">
       <always_on>true</always_on>
       <update_rate>${update_rate_imu}</update_rate>
       <visualize>true</visualize>
-      <topic>scout/imu</topic>
+      <topic>bunker/imu</topic>
     </sensor>
   </link>
   <!-- wheels -->
-  <xacro:property name="wheel_radius"     value="0.16"/>
-  <xacro:property name="wheel_width"      value="0.11"/>
-  <xacro:property name="wheel_base"       value="0.498"/>
-  <xacro:property name="wheel_separation" value="0.58306"/>
-  <xacro:macro name="wheel" params="N T X Y Z r p y">
-    <link name='${N}_wheel'>
-      <pose relative_to="chassis">${X} ${Y} ${Z} ${r} ${p} ${y}</pose>
-      <inertial auto="true">
-        <mass>8</mass>
-      </inertial>
-      <visual name='visual'>
-        <geometry>
-          <mesh><uri>meshes/wheel_type${T}.dae</uri></mesh>
-        </geometry>
-      </visual>
-      <collision name='collision'>
-        <pose relative_to="chassis">${X} ${Y} ${Z} ${((pi/2)-r)} ${p} ${y}</pose>
-        <geometry>
-          <cylinder>
-            <radius>${wheel_radius}</radius>
-            <length>${wheel_width}</length>
-          </cylinder>
-        </geometry>
-      </collision>
-    </link>
-    <joint name='${N}_wheel_joint' type='revolute'>
-      <pose relative_to='${N}_wheel'/>
-      <parent>chassis</parent>
-      <child>${N}_wheel</child>
-      <axis>
-        <xyz expressed_in='__model__'>0 1 0</xyz>
-        <limit>
-          <lower>-inf</lower>
-          <upper>inf</upper>
-        </limit>
-      </axis>
-    </joint>
-  </xacro:macro>
-  <xacro:wheel N='front_left'  T='2' X='${(wheel_base/2)}'  Y='${(wheel_separation/2)}'  Z='-0.0702' r='0.0'   p='0.0' y='0.0'/>
-  <xacro:wheel N='front_right' T='1' X='${(wheel_base/2)}'  Y='${(-wheel_separation/2)}' Z='-0.0702' r='${pi}' p='0.0' y='0.0'/>
-  <xacro:wheel N='back_left'   T='1' X='${(-wheel_base/2)}' Y='${(wheel_separation/2)}'  Z='-0.0702' r='0.0'   p='0.0' y='0.0'/>
-  <xacro:wheel N='back_right'  T='2' X='${(-wheel_base/2)}' Y='${(-wheel_separation/2)}' Z='-0.0702' r='${pi}' p='0.0' y='0.0'/>
-  <!-- visual connection -->
-  <xacro:macro name="force_bar_material">
-    <material>
-      <ambient>0.25 0.25 0.25 1.0</ambient>
-      <diffuse>0.25 0.25 0.25 1.0</diffuse>
-      <specular>0.25 0.25 0.25 1.0</specular>
-    </material>
-  </xacro:macro>
-  <xacro:macro name="force_bar_connection_visual" params="N X Y Z r p y L W H">
-    <visual name='force_bar_connection_visual_${N}'>
-      <pose relative_to="chassis">${X} ${Y} ${Z} ${r} ${p} ${y}</pose>
-      <geometry>
-        <box>
-          <size>${L} ${W} ${H}</size>
-        </box>
-      </geometry>
-      <xacro:force_bar_material/>
-    </visual>
-  </xacro:macro>
-  <link name='force_bar_connection_visual'>
-    <xacro:force_bar_connection_visual N='center_bar_left'  X='0.4'    Y='0.04'   Z='0' r='0' p='0' y='0'        L='0.2'   W='0.025' H='0.025'/>
-    <xacro:force_bar_connection_visual N='center_bar_right' X='0.4'    Y='-0.04'  Z='0' r='0' p='0' y='0'        L='0.2'   W='0.025' H='0.025'/>
-    <xacro:force_bar_connection_visual N='front_bar_top'    X='0.4875' Y='0'      Z='0' r='0' p='0' y='0'        L='0.025' W='0.41'  H='0.025'/>
-    <xacro:force_bar_connection_visual N='front_bar_left'   X='0.4575' Y='0.265'  Z='0' r='0' p='0' y='0.43633'  L='0.025' W='0.15'  H='0.025'/>
-    <xacro:force_bar_connection_visual N='front_bar_right'  X='0.4575' Y='-0.265' Z='0' r='0' p='0' y='-0.43633' L='0.025' W='0.15'  H='0.025'/>
-  </link>
-  <joint name='force_bar_connection_visual_joint' type='fixed'>
-    <pose relative_to='force_bar_connection_visual'/>
-    <parent>chassis</parent>
-    <child>force_bar_connection_visual</child>
-  </joint>
-  <!-- sensor bar -->
-  <xacro:macro name="force_bar_segment" params="P X Y Z r p y L W H">
-    <link name='force_bar_P${P}_link'>
-      <pose relative_to="chassis">${X} ${Y} ${Z} ${r} ${p} ${y}</pose>
-      <inertial auto="true">
-        <mass>1</mass>
-      </inertial>
-      <visual name='visual'>
-        <geometry>
-          <box>
-            <size>${L} ${W} ${H}</size>
-          </box>
-        </geometry>
-        <xacro:force_bar_material/>
-      </visual>
-      <collision name='collision'>
-        <geometry>
-          <box>
-            <size>${L} ${W} ${H}</size>
-          </box>
-        </geometry>
-      </collision>
-    </link>
-    <joint name='force_bar_P${P}_joint' type='fixed'>
-      <pose relative_to='force_bar_P${P}_link'/>
-      <parent>chassis</parent>
-      <child>force_bar_P${P}_link</child>
-      <sensor name='force_bar_P${P}_sensor' type='force_torque'>
-        <always_on>true</always_on>
-        <update_rate>${update_rate_force_bar}</update_rate>
-        <visualize>true</visualize>
-        <topic>/scout/force_bar/segment_${P}</topic>
-      </sensor>
-    </joint>
-  </xacro:macro>
-  <xacro:force_bar_segment P='0' X='0.466' Y='0.28'  Z='0.0' r='${pi/2}' p='0.0' y='0.43633'  L='0.005' W='0.15' H='0.14'/>
-  <xacro:force_bar_segment P='1' X='0.5'   Y='0.14'  Z='0.0' r='${pi/2}' p='0.0' y='0.0'      L='0.005' W='0.15' H='0.13'/>
-  <xacro:force_bar_segment P='2' X='0.5'   Y='0.0'   Z='0.0' r='${pi/2}' p='0.0' y='0.0'      L='0.005' W='0.15' H='0.13'/>
-  <xacro:force_bar_segment P='3' X='0.5'   Y='-0.14' Z='0.0' r='${pi/2}' p='0.0' y='0.0'      L='0.005' W='0.15' H='0.13'/>
-  <xacro:force_bar_segment P='4' X='0.466' Y='-0.28' Z='0.0' r='${pi/2}' p='0.0' y='-0.43633' L='0.005' W='0.15' H='0.14'/>
   <!-- plugins -->
   <plugin
-    filename="gz-sim-mecanum-drive-system"
-    name="gz::sim::systems::MecanumDrive">
-    <front_left_joint>front_left_wheel_joint</front_left_joint>
-    <front_right_joint>front_right_wheel_joint</front_right_joint>
-    <back_left_joint>back_left_wheel_joint</back_left_joint>
-    <back_right_joint>back_right_wheel_joint</back_right_joint>
-    <wheelbase>${wheel_base}</wheelbase>
-    <wheel_separation>${wheel_separation}</wheel_separation>
-    <wheel_radius>${wheel_radius}</wheel_radius>
-    <odom_publish_frequency>${update_rate_odom}</odom_publish_frequency>
+    filename="gz-sim-DRIVE_SYSTEM"
+    name="gz::sim::systems::DRIVE_SYSTEM">
     <topic>cmd_vel</topic>
   </plugin>
@@ -201,8 +64,4 @@
     name="gz::sim::systems::Imu">
   </plugin>
-  <plugin
-    filename="gz-sim-forcetorque-system"
-    name="gz::sim::systems::ForceTorque">
-  </plugin>
 </model>
 </sdf>

Commit message: Bunker v0.1

File: src/ros_gz_bunker_lehrforst_sim/models/bunker/model.xacro (robot description, xacro)
@@ -1,5 +1,5 @@
 <?xml version="1.0" ?>
 <sdf version="1.10" xmlns:xacro="http://ros.org/wiki/xacro">
-<model name='bunker' canonical_link='chassis'>
+<model name='bunker' canonical_link='base_link'>
   <xacro:property name="update_rate_odom"      value="1"/>
   <xacro:property name="update_rate_imu"       value="1"/>
@@ -8,6 +8,19 @@
   <xacro:property name="angular_speed"         value="0.5"/>
   <!-- base_link -->
-  <link name='chassis'>
-    <pose relative_to='__model__'>0 0 1 0 0 0</pose>
+  <link name='base_link'>
+    <pose>0.021241 0.004755 -0.127581 0 0 0</pose>
+    <inertial auto="true">
+      <mass>130</mass>
+    </inertial>
+    <visual name='visual'>
+      <geometry>
+        <mesh><uri>meshes/BUNKER.STL</uri></mesh>
+      </geometry>
+    </visual>
+    <collision name='collision'>
+      <geometry>
+        <mesh><uri>meshes/BUNKER.STL</uri></mesh>
+      </geometry>
+    </collision>
     <sensor name="imu_sensor" type="imu">
       <always_on>true</always_on>
@@ -18,10 +31,52 @@
   </link>
   <!-- wheels -->
+  <xacro:macro name="wheel" params="N m X Y Z r p y">
+    <link name="wheel${N}_Link">
+      <pose relative_to="base_link">${X} ${Y} ${Z} ${r} ${p} ${y}</pose>
+      <inertial auto="true">
+        <mass>${m}</mass>
+      </inertial>
+      <visual name='visual'>
+        <geometry>
+          <mesh><uri>meshes/wheel${N}_Link.STL</uri></mesh>
+        </geometry>
+      </visual>
+      <collision name='collision'>
+        <geometry>
+          <mesh><uri>meshes/wheel${N}_Link.STL</uri></mesh>
+        </geometry>
+      </collision>
+    </link>
+    <joint name="wheel${N}_joint" type="revolute">
+      <pose relative_to='wheel${N}_Link'/>
+      <parent>base_link</parent>
+      <child>wheel${N}_Link</child>
+      <axis>
+        <xyz>0 0 1</xyz>
+        <limit>
+          <lower>-inf</lower>
+          <upper>inf</upper>
+        </limit>
+      </axis>
+    </joint>
+  </xacro:macro>
+  <xacro:wheel N='1'   m='2' X='0.44403' Y='0.3495' Z='-0.12853' r='1.5708' p='0.0' y='-3.1416'/>
+  <xacro:wheel N='1.1' m='1' X='0.37551' Y='0.3495' Z='-0.22305' r='1.5708' p='0.0' y='-3.1416'/>
+  <xacro:wheel N='1.2' m='1' X='0.29039' Y='0.3495' Z='-0.28104' r='1.5708' p='0.0' y='-3.1416'/>
+  <xacro:wheel N='1.3' m='1' X='0.29603' Y='0.3495' Z='-0.087'   r='1.5708' p='0.0' y='-3.1416'/>
+  <xacro:wheel N='2'   m='2' X='0.44403' Y='-0.3495' Z='-0.12853' r='1.5708' p='0.0' y='-3.1416'/>
+  <xacro:wheel N='2.1' m='1' X='0.37551' Y='-0.3495' Z='-0.22305' r='1.5708' p='0.0' y='-3.1416'/>
+  <xacro:wheel N='2.2' m='1' X='0.29039' Y='-0.3495' Z='-0.28104' r='1.5708' p='0.0' y='-3.1416'/>
+  <xacro:wheel N='2.3' m='1' X='0.29603' Y='-0.3495' Z='-0.087'   r='1.5708' p='0.0' y='-3.1416'/>
+  <xacro:wheel N='3'   m='8' X='-0.38871' Y='0.295'  Z='-0.19381' r='1.5708' p='0.0' y='-3.1416'/>
+  <xacro:wheel N='3.1' m='1' X='-0.23111' Y='0.3495' Z='-0.27671' r='1.5708' p='0.0' y='-3.1416'/>
+  <xacro:wheel N='3.2' m='1' X='0.043885' Y='0.3495' Z='-0.27671' r='1.5708' p='0.0' y='-3.1416'/>
+  <xacro:wheel N='3.3' m='1' X='-0.28597' Y='0.3495' Z='-0.087'   r='1.5708' p='0.0' y='-3.1416'/>
+  <xacro:wheel N='4'   m='8' X='-0.38871' Y='-0.295'  Z='-0.19381' r='1.5708' p='0.0' y='-3.1416'/>
+  <xacro:wheel N='4.1' m='1' X='-0.23111' Y='-0.3495' Z='-0.27671' r='1.5708' p='0.0' y='-3.1416'/>
+  <xacro:wheel N='4.2' m='1' X='0.043885' Y='-0.3495' Z='-0.27671' r='1.5708' p='0.0' y='-3.1416'/>
+  <xacro:wheel N='4.3' m='1' X='-0.28597' Y='-0.3495' Z='-0.087'   r='1.5708' p='0.0' y='-3.1416'/>
   <!-- plugins -->
-  <plugin
-    filename="gz-sim-DRIVE_SYSTEM"
-    name="gz::sim::systems::DRIVE_SYSTEM">
-    <topic>cmd_vel</topic>
-  </plugin>
+  <!-- TODO: Drive System -->
   <xacro:macro name="keymap" params="D L A">
     <plugin

File: src/ros_gz_scout_lehrforst_sim/models/scout/model.xacro (robot description, xacro)
@@ -12,5 +12,5 @@
     <pose relative_to='__model__'>0 0 1 0 0 0</pose>
     <inertial auto="true">
-      <mass>50</mass>
+      <mass>67</mass>
     </inertial>
     <visual name='visual'>

Commit message: Bunker v0.2

File: src/ros_gz_bunker_lehrforst_sim/models/bunker/model.xacro (robot description, xacro)
@@ -9,5 +9,5 @@
   <!-- base_link -->
   <link name='base_link'>
-    <pose>0.021241 0.004755 -0.127581 0 0 0</pose>
+    <pose relative_to='__model__'>0 0 1 0 0 0</pose>
     <inertial auto="true">
       <mass>130</mass>
@@ -15,10 +15,28 @@
     <visual name='visual'>
       <geometry>
-        <mesh><uri>meshes/BUNKER.STL</uri></mesh>
+        <mesh><uri>meshes/base_link.STL</uri></mesh>
       </geometry>
+      <material>
+        <ambient>0.25 0.25 0.25 1.0</ambient>
+        <diffuse>0.25 0.25 0.25 1.0</diffuse>
+        <specular>0.25 0.25 0.25 1.0</specular>
+      </material>
+    </visual>
+    <visual name='visual2'>
+      <geometry>
+        <mesh><uri>meshes/base2_Link.STL</uri></mesh>
+      </geometry>
+      <material>
+        <ambient>0.75 0.75 0.75 1.0</ambient>
+        <diffuse>0.75 0.75 0.75 1.0</diffuse>
+        <specular>0.75 0.75 0.75 1.0</specular>
+      </material>
     </visual>
     <collision name='collision'>
+      <pose>0 0 -0.15 0 0 0</pose>
       <geometry>
-        <mesh><uri>meshes/BUNKER.STL</uri></mesh>
+        <box>
+          <size>0.95 0.4 0.2</size>
+        </box>
       </geometry>
     </collision>
@@ -31,5 +49,5 @@
   </link>
   <!-- wheels -->
-  <xacro:macro name="wheel" params="N m X Y Z r p y">
+  <xacro:macro name="wheel" params="N m R W P X Y Z r p y">
     <link name="wheel${N}_Link">
       <pose relative_to="base_link">${X} ${Y} ${Z} ${r} ${p} ${y}</pose>
@@ -38,11 +56,21 @@
       </inertial>
       <visual name='visual'>
+        <pose relative_to="base_link">${X} ${Y+P} ${Z} ${r} ${p} ${y}</pose>
         <geometry>
           <mesh><uri>meshes/wheel${N}_Link.STL</uri></mesh>
         </geometry>
+        <material>
+          <ambient>0.5 0.5 0.5 1.0</ambient>
+          <diffuse>0.5 0.5 0.5 1.0</diffuse>
+          <specular>0.5 0.5 0.5 1.0</specular>
+        </material>
       </visual>
       <collision name='collision'>
+        <pose relative_to="base_link">${X} ${Y+P} ${Z} ${r} ${p} ${y}</pose>
         <geometry>
-          <mesh><uri>meshes/wheel${N}_Link.STL</uri></mesh>
+          <cylinder>
+            <radius>${R}</radius>
+            <length>${W}</length>
+          </cylinder>
         </geometry>
       </collision>
@@ -61,20 +89,20 @@
     </joint>
   </xacro:macro>
-  <xacro:wheel N='1'   m='2' X='0.44403' Y='0.3495' Z='-0.12853' r='1.5708' p='0.0' y='-3.1416'/>
-  <xacro:wheel N='1.1' m='1' X='0.37551' Y='0.3495' Z='-0.22305' r='1.5708' p='0.0' y='-3.1416'/>
-  <xacro:wheel N='1.2' m='1' X='0.29039' Y='0.3495' Z='-0.28104' r='1.5708' p='0.0' y='-3.1416'/>
-  <xacro:wheel N='1.3' m='1' X='0.29603' Y='0.3495' Z='-0.087'   r='1.5708' p='0.0' y='-3.1416'/>
-  <xacro:wheel N='2'   m='2' X='0.44403' Y='-0.3495' Z='-0.12853' r='1.5708' p='0.0' y='-3.1416'/>
-  <xacro:wheel N='2.1' m='1' X='0.37551' Y='-0.3495' Z='-0.22305' r='1.5708' p='0.0' y='-3.1416'/>
-  <xacro:wheel N='2.2' m='1' X='0.29039' Y='-0.3495' Z='-0.28104' r='1.5708' p='0.0' y='-3.1416'/>
-  <xacro:wheel N='2.3' m='1' X='0.29603' Y='-0.3495' Z='-0.087'   r='1.5708' p='0.0' y='-3.1416'/>
-  <xacro:wheel N='3'   m='8' X='-0.38871' Y='0.295'  Z='-0.19381' r='1.5708' p='0.0' y='-3.1416'/>
-  <xacro:wheel N='3.1' m='1' X='-0.23111' Y='0.3495' Z='-0.27671' r='1.5708' p='0.0' y='-3.1416'/>
-  <xacro:wheel N='3.2' m='1' X='0.043885' Y='0.3495' Z='-0.27671' r='1.5708' p='0.0' y='-3.1416'/>
-  <xacro:wheel N='3.3' m='1' X='-0.28597' Y='0.3495' Z='-0.087'   r='1.5708' p='0.0' y='-3.1416'/>
-  <xacro:wheel N='4'   m='8' X='-0.38871' Y='-0.295'  Z='-0.19381' r='1.5708' p='0.0' y='-3.1416'/>
-  <xacro:wheel N='4.1' m='1' X='-0.23111' Y='-0.3495' Z='-0.27671' r='1.5708' p='0.0' y='-3.1416'/>
-  <xacro:wheel N='4.2' m='1' X='0.043885' Y='-0.3495' Z='-0.27671' r='1.5708' p='0.0' y='-3.1416'/>
-  <xacro:wheel N='4.3' m='1' X='-0.28597' Y='-0.3495' Z='-0.087'   r='1.5708' p='0.0' y='-3.1416'/>
+  <xacro:wheel N='1'   R='0.05'  W='0.05' P='-0.075' m='2' X='0.44403'  Y='0.3495'  Z='-0.12853' r='1.5708' p='0.0' y='-3.1416'/>
+  <xacro:wheel N='1.1' R='0.04'  W='0.05' P='-0.075' m='1' X='0.37551'  Y='0.3495'  Z='-0.22305' r='1.5708' p='0.0' y='-3.1416'/>
+  <xacro:wheel N='1.2' R='0.05'  W='0.05' P='-0.075' m='1' X='0.29039'  Y='0.3495'  Z='-0.28104' r='1.5708' p='0.0' y='-3.1416'/>
+  <xacro:wheel N='1.3' R='0.05'  W='0.05' P='-0.075' m='1' X='0.29603'  Y='0.3495'  Z='-0.087'   r='1.5708' p='0.0' y='-3.1416'/>
+  <xacro:wheel N='2'   R='0.05'  W='0.05' P='0.075'  m='2' X='0.44403'  Y='-0.3495' Z='-0.12853' r='1.5708' p='0.0' y='-3.1416'/>
+  <xacro:wheel N='2.1' R='0.04'  W='0.05' P='0.075'  m='1' X='0.37551'  Y='-0.3495' Z='-0.22305' r='1.5708' p='0.0' y='-3.1416'/>
+  <xacro:wheel N='2.2' R='0.05'  W='0.05' P='0.075'  m='1' X='0.29039'  Y='-0.3495' Z='-0.28104' r='1.5708' p='0.0' y='-3.1416'/>
+  <xacro:wheel N='2.3' R='0.05'  W='0.05' P='0.075'  m='1' X='0.29603'  Y='-0.3495' Z='-0.087'   r='1.5708' p='0.0' y='-3.1416'/>
+  <xacro:wheel N='3'   R='0.075' W='0.05' P='0'      m='8' X='-0.38871' Y='0.295'   Z='-0.19381' r='1.5708' p='0.0' y='-3.1416'/>
+  <xacro:wheel N='3.1' R='0.05'  W='0.05' P='-0.075' m='1' X='-0.23111' Y='0.3495'  Z='-0.27671' r='1.5708' p='0.0' y='-3.1416'/>
+  <xacro:wheel N='3.2' R='0.05'  W='0.05' P='-0.075' m='1' X='0.043885' Y='0.3495'  Z='-0.27671' r='1.5708' p='0.0' y='-3.1416'/>
+  <xacro:wheel N='3.3' R='0.05'  W='0.05' P='-0.075' m='1' X='-0.28597' Y='0.3495'  Z='-0.087'   r='1.5708' p='0.0' y='-3.1416'/>
+  <xacro:wheel N='4'   R='0.075' W='0.05' P='0'      m='8' X='-0.38871' Y='-0.295'  Z='-0.19381' r='1.5708' p='0.0' y='-3.1416'/>
+  <xacro:wheel N='4.1' R='0.05'  W='0.05' P='0.075'  m='1' X='-0.23111' Y='-0.3495' Z='-0.27671' r='1.5708' p='0.0' y='-3.1416'/>
+  <xacro:wheel N='4.2' R='0.05'  W='0.05' P='0.075'  m='1' X='0.043885' Y='-0.3495' Z='-0.27671' r='1.5708' p='0.0' y='-3.1416'/>
+  <xacro:wheel N='4.3' R='0.05'  W='0.05' P='0.075'  m='1' X='-0.28597' Y='-0.3495' Z='-0.087'   r='1.5708' p='0.0' y='-3.1416'/>
   <!-- plugins -->
   <!-- TODO: Drive System -->

Commit message: Bunker v0.3 (added drive system draft)

File: src/ros_gz_bunker_lehrforst_sim/models/bunker/model.xacro (robot description, xacro)
@@ -4,7 +4,7 @@
   <xacro:property name="update_rate_odom"      value="1"/>
   <xacro:property name="update_rate_imu"       value="1"/>
-  <xacro:property name="update_rate_pose"      value="3"/>
-  <xacro:property name="linear_speed"          value="0.5"/>
-  <xacro:property name="angular_speed"         value="0.5"/>
+  <xacro:property name="update_rate_pose"      value="1"/>
+  <xacro:property name="linear_speed"          value="1"/>
+  <xacro:property name="angular_speed"         value="1"/>
   <!-- base_link -->
   <link name='base_link'>
@@ -106,5 +106,26 @@
   <xacro:wheel N='4.3' R='0.05'  W='0.05' P='0.075'  m='1' X='-0.28597' Y='-0.3495' Z='-0.087'   r='1.5708' p='0.0' y='-3.1416'/>
   <!-- plugins -->
-  <!-- TODO: Drive System -->
+  <plugin
+    filename="gz-sim-diff-drive-system"
+    name="gz::sim::systems::DiffDrive">
+    <left_joint>wheel1_joint</left_joint>
+    <left_joint>wheel1.1_joint</left_joint>
+    <left_joint>wheel1.2_joint</left_joint>
+    <left_joint>wheel1.3_joint</left_joint>
+    <left_joint>wheel3_joint</left_joint>
+    <left_joint>wheel3.1_joint</left_joint>
+    <left_joint>wheel3.2_joint</left_joint>
+    <left_joint>wheel3.3_joint</left_joint>
+    <right_joint>wheel2_joint</right_joint>
+    <right_joint>wheel2.1_joint</right_joint>
+    <right_joint>wheel2.2_joint</right_joint>
+    <right_joint>wheel2.3_joint</right_joint>
+    <right_joint>wheel4_joint</right_joint>
+    <right_joint>wheel4.1_joint</right_joint>
+    <right_joint>wheel4.2_joint</right_joint>
+    <right_joint>wheel4.3_joint</right_joint>
+    <odom_publish_frequency>${update_rate_odom}</odom_publish_frequency>
+    <topic>cmd_vel</topic>
+  </plugin>
   <xacro:macro name="keymap" params="D L A">
     <plugin
